File: hw/kicad/11ua/11ua.sch (KiCad schematic (older format))
At the start: 26 parts, among them J1 RJ45_LED, J2 RJ45_LED, J3 CONN_01X04, J4 CONN_01X04, U1 OPA4376

Commit message: added IKCM30F60GD
Parts:
- removed C1, C2, C3, C4, C7, C8: 27p, stmbl-kicad-lib:C_0603, symbol stmbl:C
- removed C10, C11, C12: C, stmbl-kicad-lib:C_0603, symbol stmbl:C
- removed C13, C14: CP, Capacitor_Tantalum_SMD:CP_EIA-2012-15_AVX-P, symbol Device:CP
- removed C5, C6: 100n, stmbl-kicad-lib:C_0603, symbol stmbl:C
- removed J1, J2: RJ45_LED, stmbl:RJ45_LED, symbol stmbl:RJ45_LED
- removed J3, J4: CONN_01X04, stmbl:RM3.81_1x4_UP, symbol stmbl:CONN_01X04
- removed R1, R10, R2, R3, R4, R9: 100k, stmbl-kicad-lib:R_0603, symbol stmbl:R
- removed R7, R8: 120, stmbl-kicad-lib:R_0603, symbol stmbl:R
- removed U1: OPA4376, Housings_SSOP:TSSOP-14_4.4x5mm_Pitch0.65mm, symbol Amplifier_Operational:OPA4376
Connections:
- net labels removed: +5V, 2.5V, GND
- wire segments 157 -> 0
